File: NixiePower.brd (EAGLE design)
At the start: 66 x 38.7 mm, 21 parts, among them IC1 MC34063AD, T1 MJD31

Commit message: Commit of Rev.C version
Parts:
- removed C5, C6: 470nF, rcl:C1206K
- removed D1, D2: MURS120, diode:DO214AA
- removed T1: MJD31, transistor:DPAK
- added IC3: IRS44273L, own-collection:SOT23-5
- added Q1: IRF740D2PAK, own-collection:D2PAK
- added R6: 0.75, rcl-2:R1206
- added R7: 20, rcl-2:R1206
- added R8: 0, rcl-2:R1206
- C2: value 400pF -> 470pF
- C4: value 470nF -> 0.1uF
- L1: value DR125 -> 220uH
- R1: value 0.5 -> 0.75
- R2: value 180 -> 20k; device rcl-2:R1206 -> rcl:RTRIM4G/J
- R3: value 47k -> 560k
- R4: value 2.2k -> 3.3k
- R5: value (none) -> 1.5k
- moved R2 23.8 mm to (18.7, 23.2)
- moved C4 20.1 mm to (48.9, 21.9), turned to 90 degrees
- moved D3 6.99 mm to (14.0, 10.2), turned to 0 degrees
- moved R5 6.38 mm to (50.2, 13.7)
- moved R3 5.41 mm to (15.9, 29.5), turned to 90 degrees
- moved R4 5.41 mm to (15.9, 16.8), turned to 90 degrees
- moved L1 3.62 mm to (30.2, 23.2)
- moved R1 3.13 mm to (48.9, 31.1)
- moved C2 2.03 mm to (50.2, 17.1)
- moved C3 0.71 mm to (8.57, 30.5)
Connections:
- new net N$6: C3.+, D3.C, PAD3.1, R3.2
- new net VCC: C1.+, IC1.6, IC1.8, PAD1.1, R1.1, R6.1, R8.1
- net GND: now also C4.1, IC3.2, Q1.3; no longer C5.2, C6.2, T1.3
- net N$1: now also D3.A, Q1.4; no longer C4.2, D1.A, IC1.1, T1.4
- net N$10: now also R2.3, R4.2; no longer C3.+, C6.1, D3.C, PAD3.1, R3.2
- net N$11: now also IC3.1; no longer T1.1
- net N$3: now also R6.2; no longer R2.1
- net N$4: now also IC1.1, IC3.5, R8.2; no longer IC1.8, R2.2
- net N$5: now also Q1.1, R7.2; no longer C1.+, IC1.6, PAD1.1, R1.1
- net N$7: now also C4.2, R2.2; no longer R3.1, R4.2
- net N$8: now also IC3.3, IC3.4, R7.1; no longer C5.1, D1.C, D2.A
- net N$9: now also R2.1, R3.1; no longer C4.1, D2.C, D3.A
Routing:
- net GND: track 78.7 -> 156.5 mm
- net N$10: track 46.1 -> 3.89 mm
- net VCC: track 0.00 -> 31.4 mm
- net N$6: track 0.00 -> 31.3 mm
- net N$1: track 38.9 -> 17.9 mm
- net N$5: track 21.6 -> 4.93 mm
- net N$3: track 20.4 -> 29.5 mm
- net N$9: track 10.2 -> 3.89 mm
- net N$4: track 4.02 -> 10.3 mm
- net N$11: track 11.0 -> 13.9 mm
- net N$7: track 34.1 -> 31.2 mm
- net N$8: track 10.6 -> 8.35 mm
- added copper zone on layer 1, net N$6
- removed copper zone on layer 1, net N$10
- removed copper zone on layer 1, net N$5

Commit message: Commit of the current version
Parts:
- added D1: MURS120, diode:DO214AA
Connections:
- new net N$12: D1.A, PAD1.1
- net VCC: now also D1.C; no longer PAD1.1
Routing:
- net VCC: track 31.4 -> 24.7 mm
- net N$12: track 0.00 -> 2.53 mm
Changed lines of the file:
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@@
 <element name="R2" library="rcl" package="RTRIM4G/J" value="20k" x="18.7325" y="23.1775" rot="R270"/>
 <element name="Q1" library="own-collection" package="D2PAK" value="IRF740D2PAK" x="29.2975" y="10.16" rot="R90"/>
+<element name="D1" library="diode" package="DO214AA" value="MURS120" x="53.34" y="31.115" rot="R90"/>
 </elements>
 <signals>
@@
 <contactref element="R6" pad="1"/>
 <contactref element="C1" pad="+"/>
-<contactref element="PAD1" pad="1"/>
-<wire x1="53.34" y1="26.035" x2="53.34" y2="29.693" width="2.1844" layer="1"/>
-<wire x1="53.34" y1="29.693" x2="53.34" y2="36.195" width="2.1844" layer="1"/>
 <wire x1="46.355" y1="29.693" x2="48.895" y2="29.693" width="1.27" layer="1"/>
 <wire x1="45.085" y1="24.825" x2="45.085" y2="28.423" width="0.6096" layer="1"/>
 <wire x1="45.085" y1="28.423" x2="46.355" y2="29.693" width="0.6096" layer="1"/>
-<wire x1="53.34" y1="29.693" x2="48.895" y2="29.693" width="1.27" layer="1"/>
 <contactref element="IC1" pad="8"/>
 <contactref element="IC1" pad="6"/>
@@
 <wire x1="44.45" y1="22.86" x2="45.085" y2="23.495" width="0.6096" layer="1"/>
 <wire x1="45.085" y1="23.495" x2="45.085" y2="24.825" width="0.6096" layer="1"/>
+<contactref element="D1" pad="C"/>
+<wire x1="53.34" y1="28.565" x2="53.34" y2="27.305" width="1.4224" layer="1"/>
+<wire x1="53.34" y1="27.305" x2="53.34" y2="26.035" width="1.4224" layer="1"/>
+<wire x1="48.895" y1="29.693" x2="51.283" y2="27.305" width="1.27" layer="1"/>
+<wire x1="51.283" y1="27.305" x2="53.34" y2="27.305" width="1.27" layer="1"/>
 </signal>
 <signal name="N$5">
@@
 <wire x1="15.875" y1="22.0275" x2="15.9825" y2="22.0275" width="0.4064" layer="1"/>
 </signal>
+<signal name="N$12">
+<contactref element="PAD1" pad="1"/>
+<contactref element="D1" pad="A"/>
+<wire x1="53.34" y1="33.665" x2="53.34" y2="36.195" width="1.4224" layer="1"/>
+</signal>
 </signals>
