File: NixiePower.sch (EAGLE design)
At the start: 14 parts, among them IC1 MC34063AD

Commit message: Commit of Rev.B version
Parts:
- added C4, C5, C6: 470nF, rcl:C-EUC1206K
- added D1, D2: MURS120, diode:DIODE-DO214AA
- added R5: (no value), rcl-2:R-EU_R1206
- added T1: MJD31, transistor:MJD31
Connections:
- removed net N$6: C3.+, D3.C, PAD3.P, R3.2
- new net N$10: C3.+, C6.1, D3.C, PAD3.P, R3.2
- new net N$11: IC1.SWE, R5.2, T1.B
- new net N$8: C5.1, D1.C, D2.A
- new net N$9: C4.1, D2.C, D3.A
- net GND: now also C5.2, C6.2, R5.1, T1.E; no longer IC1.SWE
- net N$1: now also C4.2, D1.A, T1.C; no longer D3.A
Other:
- moved on the sheet: C3, D3, PAD3, PAD4

Commit message: Commit of Rev.C version
Parts:
- removed C5, C6: 470nF, rcl:C-EUC1206K
- removed D1, D2: MURS120, diode:DIODE-DO214AA
- removed T1: MJD31, transistor:MJD31
- added IC3: IRS44273L, own-collection:IRS44273L
- added Q1: IRF740D2PAK, own-collection:IRF740D2PAK
- added R6: 0.75, rcl-2:R-EU_R1206
- added R7: 20, rcl-2:R-EU_R1206
- added R8: 0, rcl-2:R-EU_R1206
- C2: value 400pF -> 470pF
- C4: value 470nF -> 0.1uF
- L1: value DR125 -> 220uH
- R1: value 0.5 -> 0.75
- R2: value 180 -> 20k; device rcl-2:R-EU_R1206 -> rcl:R-TRIMM4G/J
- R3: value 47k -> 560k
- R4: value 2.2k -> 3.3k
- R5: value (none) -> 1.5k
Connections:
- new net N$6: C3.+, D3.C, PAD3.P, R3.2
- new net VCC: C1.+, IC1.DC, IC1.VCC, PAD1.P, R1.1, R6.1, R8.1
- net GND: now also C4.1, IC3.COM, Q1.S; no longer C5.2, C6.2, T1.E
- net N$1: now also D3.A, Q1.D; no longer C4.2, D1.A, IC1.SWC, T1.C
- net N$10: now also R2.E, R4.2; no longer C3.+, C6.1, D3.C, PAD3.P, R3.2
- net N$11: now also IC3.IN; no longer T1.B
- net N$3: now also R6.2; no longer R2.1
- net N$4: now also IC1.SWC, IC3.VCC, R8.2; no longer IC1.DC, R2.2
- net N$5: now also Q1.G, R7.2; no longer C1.+, IC1.VCC, PAD1.P, R1.1
- net N$7: now also C4.2, R2.S; no longer R3.1, R4.2
- net N$8: now also IC3.OUT1, IC3.OUT2, R7.1; no longer C5.1, D1.C, D2.A
- net N$9: now also R2.A, R3.1; no longer C4.1, D2.C, D3.A
Other:
- moved on the sheet: C1, C3, C4, D3, L1, PAD1, PAD2, PAD3, PAD4, R1, R3, R4

Commit message: Commit of the current version
Parts:
- added D1: MURS120, diode:DIODE-DO214AA
Connections:
- new net N$12: D1.A, PAD1.P
- net VCC: now also D1.C; no longer PAD1.P
Other:
- moved on the sheet: PAD1, PAD2
Changed lines of the file:
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@@
 <part name="R2" library="rcl" deviceset="R-TRIMM" device="4G/J" value="20k"/>
 <part name="Q1" library="own-collection" deviceset="IRF740" device="D2PAK" value="IRF740D2PAK"/>
+<part name="D1" library="diode" deviceset="DIODE-" device="DO214AA" value="MURS120"/>
 </parts>
 <sheets>
@@
 <instance part="R4" gate="G$1" x="66.04" y="17.78" rot="R90"/>
 <instance part="GND5" gate="1" x="66.04" y="7.62"/>
-<instance part="PAD1" gate="1" x="-10.16" y="55.88"/>
-<instance part="PAD2" gate="1" x="-10.16" y="48.26"/>
-<instance part="GND6" gate="1" x="0" y="43.18"/>
+<instance part="PAD1" gate="1" x="-17.78" y="55.88"/>
+<instance part="PAD2" gate="1" x="-17.78" y="48.26"/>
+<instance part="GND6" gate="1" x="-5.08" y="43.18"/>
 <instance part="PAD3" gate="1" x="208.28" y="78.74" rot="R180"/>
 <instance part="PAD4" gate="1" x="208.28" y="58.42" rot="R180"/>
@@
 <instance part="GND12" gate="1" x="165.1" y="40.64"/>
 <instance part="P+3" gate="VCC" x="38.1" y="66.04"/>
-<instance part="P+5" gate="VCC" x="0" y="60.96"/>
+<instance part="P+5" gate="VCC" x="-5.08" y="63.5"/>
 <instance part="R8" gate="G$1" x="86.36" y="68.58" rot="R270"/>
 <instance part="P+4" gate="VCC" x="86.36" y="76.2"/>
@@
 <instance part="R2" gate="G$1" x="66.04" y="30.48" rot="R180"/>
 <instance part="Q1" gate="G$1" x="162.56" y="50.8"/>
+<instance part="D1" gate="G$1" x="-10.16" y="55.88" smashed="yes">
+<attribute name="NAME" x="-12.7" y="58.9026" size="1.778" layer="95"/>
+<attribute name="VALUE" x="-12.7" y="51.0286" size="1.778" layer="96"/>
+</instance>
 </instances>
 <busses>
@@
 <pinref part="PAD2" gate="1" pin="P"/>
 <pinref part="GND6" gate="1" pin="GND"/>
-<wire x1="-7.62" y1="48.26" x2="0" y2="48.26" width="0.1524" layer="91"/>
-<wire x1="0" y1="48.26" x2="0" y2="45.72" width="0.1524" layer="91"/>
+<wire x1="-15.24" y1="48.26" x2="-5.08" y2="48.26" width="0.1524" layer="91"/>
+<wire x1="-5.08" y1="48.26" x2="-5.08" y2="45.72" width="0.1524" layer="91"/>
 </segment>
 <segment>
@@
 </segment>
 <segment>
-<pinref part="PAD1" gate="1" pin="P"/>
-<pinref part="P+5" gate="VCC" pin="VCC"/>
-<wire x1="-7.62" y1="55.88" x2="0" y2="55.88" width="0.1524" layer="91"/>
-<wire x1="0" y1="55.88" x2="0" y2="58.42" width="0.1524" layer="91"/>
-</segment>
-<segment>
 <pinref part="IC1" gate="G$1" pin="DC"/>
 <pinref part="P+3" gate="VCC" pin="VCC"/>
@@
 <pinref part="P+4" gate="VCC" pin="VCC"/>
 </segment>
+<segment>
+<pinref part="D1" gate="G$1" pin="C"/>
+<pinref part="P+5" gate="VCC" pin="VCC"/>
+<wire x1="-7.62" y1="55.88" x2="-5.08" y2="55.88" width="0.1524" layer="91"/>
+<wire x1="-5.08" y1="55.88" x2="-5.08" y2="60.96" width="0.1524" layer="91"/>
+</segment>
 </net>
 <net name="N$5" class="0">
@@
 </segment>
 </net>
+<net name="N$12" class="0">
+<segment>
+<pinref part="PAD1" gate="1" pin="P"/>
+<pinref part="D1" gate="G$1" pin="A"/>
+<wire x1="-15.24" y1="55.88" x2="-12.7" y2="55.88" width="0.1524" layer="91"/>
+</segment>
+</net>
